File: kicad_project/santas_sequencer.kicad_pcb (KiCad board)
At the start: 2 copper layers, 94.8 x 56 mm, 41 parts, among them Q1 BC847, Q2 BC847, SW1 SW_DPDT_x2, U1 CD4017

Commit message: Updating the pcb to correct a project flaw: the transistors ground plane was isolated from other grounds
Routing:
- net GND: vias 2 -> 3
